Commit message: URDF II

File: src/Grete_r2d2/urdf/r2d2.urdf.xacro (robot description, xacro)
@@ -10,5 +10,4 @@
   <xacro:property name="length_lens" value="0.04" />
   <xacro:property name="radius_lens" value="0.03" />
-<!--COLOURS-->
   <material name="blue">
     <color rgba="0 0 0.8 1"/>
@@ -20,5 +19,4 @@
     <color rgba="1 1 1 1"/>
   </material>
-<!--MACROS-->
   <xacro:macro name="default_inertial" params="mass">
     <inertial>
@@ -27,5 +25,4 @@
     </inertial>
   </xacro:macro>
-<!--PARTS-->
   <link name="base_link">
     <visual>
@@ -42,4 +39,11 @@
     <xacro:default_inertial mass="10"/>
   </link>
+  <link name="base_footprint">
+  </link>
+  <joint name="joint_base_footprint" type="fixed">
+    <parent link="base_footprint"/>
+    <child link="base_link"/>
+    <origin xyz="0 0 ${wheeldiam+bodylen/2+0.1}"/>
+  </joint>
   <xacro:macro name="wheel" params="prefix suffix reflect">
     <link name="${prefix}_${suffix}_wheel">

Commit message: Assignment III

File: src/Grete_r2d2/urdf/r2d2.urdf.xacro (robot description, xacro)
@@ -248,3 +248,80 @@
     <origin rpy="0 0 0" xyz="${length_lens-.04} 0 0"/>
   </joint>
+  <link name="base_scan">
+    <visual>
+      <origin xyz="0 0 0" rpy="0 0 0"/>
+      <geometry>
+        <mesh filename="package://turtlebot3_description/meshes/sensors/lds.stl" scale="0.001 0.001 0.001"/>
+      </geometry>
+      <material name="black"/>
+    </visual>
+    <collision>
+      <origin xyz="0.015 0 -0.0065" rpy="0 0 0"/>
+      <geometry>
+        <cylinder length="0.0315" radius="0.055"/>
+      </geometry>
+    </collision>
+    <inertial>
+      <mass value="0.114" />
+      <origin xyz="0 0 0" />
+      <inertia ixx="0.001" ixy="0.0" ixz="0.0"
+               iyy="0.001" iyz="0.0"
+               izz="0.001" />
+    </inertial>
+  </link>
+  <joint name="joint_base_scan" type="fixed">
+    <parent link="base_footprint"/>
+    <child link="base_scan"/>
+    <origin xyz="${width-0.04} 0 ${wheeldiam+bodylen+width+0.0975}" rpy="0 0 0"/>
+  </joint>
+  <gazebo reference="base_scan">
+    <material>Gazebo/FlatBlack</material>
+    <sensor type="ray" name="lds_lfcd_sensor">
+      <pose>0 0 0 0 0 0</pose>
+      <visualize>false</visualize>
+      <update_rate>5</update_rate>
+      <ray>
+        <scan>
+          <horizontal>
+            <samples>360</samples>
+            <resolution>1</resolution>
+            <min_angle>0.0</min_angle>
+            <max_angle>6.28319</max_angle>
+          </horizontal>
+        </scan>
+        <range>
+          <min>0.120</min>
+          <max>3.5</max>
+          <resolution>0.015</resolution>
+        </range>
+        <noise>
+          <type>gaussian</type>
+          <mean>0.0</mean>
+          <stddev>0.01</stddev>
+        </noise>
+      </ray>
+      <plugin name="gazebo_ros_lds_lfcd_controller" filename="libgazebo_ros_laser.so">
+        <topicName>scan</topicName>
+        <frameName>base_scan</frameName>
+      </plugin>
+    </sensor>
+  </gazebo>
+  <gazebo>
+    <plugin name="skid_steer_drive_controller" filename="libgazebo_ros_skid_steer_drive.so">
+	<alwaysOn>true</alwaysOn>
+	<updateRate>50.0</updateRate>
+	<leftFrontJoint>left_front_wheel_joint</leftFrontJoint>
+	<rightFrontJoint>right_front_wheel_joint</rightFrontJoint>
+	<leftRearJoint>left_back_wheel_joint</leftRearJoint>
+	<rightRearJoint>right_back_wheel_joint</rightRearJoint>
+	<wheelSeparation>${2.0*baselen/3.0}</wheelSeparation>
+	<wheelDiameter>${wheeldiam}</wheelDiameter>
+	<torque>10</torque>
+	<broadcastTF>1</broadcastTF>
+	<odometryFrame>odom</odometryFrame>
+	<commandTopic>cmd_vel</commandTopic>
+	<odometryTopic>/odom</odometryTopic>
+	<robotBaseFrame>base_footprint</robotBaseFrame>
+    </plugin>
+  </gazebo>
 </robot>
